File: IP6822_EVA_Board/IP6822_EVA_Board.kicad_sch (KiCad schematic)
At the start: 2 parts, among them U1 IP6822

Commit message: Finished EVA_Board
Parts:
- added C10, C11, C8, C9: 10nF, Capacitor_SMD:C_0603_1608Metric, symbol Device:C
- added C12: 2.2uF, Capacitor_SMD:C_0603_1608Metric, symbol Device:C
- added C2, C3: 22uF, Capacitor_SMD:C_0603_1608Metric, symbol Device:C
- added C4, C5, C6, C7: 0.1uF, Capacitor_SMD:C_0805_2012Metric, symbol Device:C
- added D1: 1N5819WS, Diode_SMD:D_SOD-323, symbol Diode:1N5819WS
- added J1: USB_C_Receptacle, Connector_USB:USB_C_Receptacle_HCTL_HC-TYPE-C-16P-01A, symbol Connector:USB_C_Receptacle
- added L1: 6.3uH, Inductor_SMD:L_2010_5025Metric, symbol Device:L
- added L2: 0R, Inductor_SMD:L_0805_2012Metric, symbol Device:L
- added Q1, Q2: IRF7389PBF, SOIC127P600X175-8N, symbol SamacSys_Parts:IRF7389PBF
- added R1, R2, R3, R4: 10K, Resistor_SMD:R_0603_1608Metric, symbol Device:R
- added R10, R7: 33K, Resistor_SMD:R_0603_1608Metric, symbol Device:R
- added R11, R12: 22R, Resistor_SMD:R_0603_1608Metric, symbol Device:R
- added R13, R14: 0R, Resistor_SMD:R_0603_1608Metric, symbol Device:R
- added R5: 20mR, Resistor_SMD:R_1206_3216Metric, symbol Device:R
- added R6, R8, R9: 3K3, Resistor_SMD:R_0603_1608Metric, symbol Device:R
- added TP1, TP2, TP3, TP4, TP5, TP6, TP7, TP8, TP9: TestPoint, TestPoint:TestPoint_Bridge_Pitch3.81mm_Drill1.3mm, symbol Connector:TestPoint
- added Z1: MMSZ5244A, MMSZ5252B, symbol SamacSys_Parts:MMSZ5244A
- C1: footprint (none) -> Capacitor_SMD:C_0603_1608Metric
Connections:
- net DRV1H: now also R13.2, R2.1, TP1.1
- net DRV1L: now also R1.1, TP2.1
- net DRV2H: now also R14.1, R3.1, TP3.1
- net DRV2L: now also R4.1, TP4.1
- net GND: now also C10.1, C11.1, C12.1, C8.1, J1.A1 (GND), J1.A12 (GND), J1.B1 (GND), J1.B12 (GND), J1.S1 (SHIELD), L2.1, R5.1, R7.1, R9.2, TP9.1, Z1.2 (A)
- net ISENSE: now also C8.2, R6.2
- net USB_CC1: now also J1.A5 (CC1)
- net USB_CC2: now also J1.B5 (CC2)
- net USB_DN: now also R11.2
- net USB_DP: now also R12.2
- net VBUS: now also C2.2, C3.2, J1.A4 (VBUS), J1.A9 (VBUS), J1.B4 (VBUS), J1.B9 (VBUS), Q1.3 (S2), Q2.3 (S2), R13.1, R14.2, TP8.1, Z1.1 (K)
- net VCOIL: now also C11.2, R10.1, R9.1, TP6.1
- net VDEM: now also C9.1, TP7.1
- net VCC: no longer names the net of U1.6 (VCC)
- net VCC: now also C12.2
- new net: Q2.2 (G1), R4.2
- new net: C4.2, C5.2, C6.2, C7.2, Q2.5 (D_1), Q2.6 (D_2), Q2.7 (D_3), Q2.8 (D_4)
- new net: C10.2, C9.2, R7.2, R8.2
- new net: L1.1, Q1.5 (D_1), Q1.6 (D_2), Q1.7 (D_3), Q1.8 (D_4)
- new net: J1.A6 (D+), J1.B6 (D+), R12.1
- new net: J1.A7 (D-), J1.B7 (D-), R11.1
- new net: D1.1 (K), R10.2, R8.1
- new net: Q2.4 (G2), R3.2
- new net: Q1.2 (G1), R1.2
- new net: Q1.4 (G2), R2.2
- new net GNDPWR: C2.1, C3.1, L2.2, Q1.1 (S1), Q2.1 (S1), R5.2, R6.1
- new net VC: C4.1, C5.1, C6.1, C7.1, D1.2 (A), L1.2, TP5.1
- no-connect marks 0 -> 10
